File: output/pcbs/p48v2.kicad_pcb (KiCad board)
At the start: 2 copper layers, 255 x 72 mm, 160 parts

Commit message: Save PCB state (locked - no more ergogen regeneration)
Parts:
- moved D49 13.1 mm to (339.7, -66.0), turned to 90 degrees
- moved R1 8.45 mm to (338.9, -73.6), turned to -90 degrees
- moved R2 8.41 mm to (338.9, -77.4), turned to 90 degrees
- moved H10 7.20 mm to (347.2, -84.3)
- moved J1 6.95 mm to (345.9, -74.7)
- moved 19.051 1.00 mm to (323.5, -60.5)
- moved H11 0.36 mm to (340.3, -17.7)
- moved H1 0.28 mm to (90.7, -84.3)
- moved H3 0.28 mm to (90.7, -17.7)
- moved H2 0.22 mm to (305.4, -84.3)
- moved H4 0.22 mm to (305.4, -17.7)
- moved D24 0.22 mm to (188.9, -85.8)
- moved D28 0.22 mm to (206.9, -85.8)
- moved H9 0.22 mm to (197.9, -17.7)
- moved D40 0.20 mm to (261.0, -85.8)
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Connections:
- LED1 pad 2: LED48 -> LED37
- LED1 pad 4: LED47 -> LED36
- LED10 pad 2: LED27 -> LED34
- LED10 pad 4: LED26 -> LED33
- LED11 pad 2: LED22 -> LED15
- LED11 pad 4: LED21 -> LED14
- LED12 pad 2: LED3 -> LED10
- LED12 pad 4: LED2 -> LED9
- LED13 pad 2: LED45 -> LED40
- LED13 pad 4: LED44 -> LED39
- LED14 pad 2: LED28 -> LED33
- LED14 pad 4: LED27 -> LED32
- LED15 pad 2: LED21 -> LED16
- LED15 pad 4: LED20 -> LED15
- LED16 pad 2: LED4 -> LED9
- LED16 pad 4: LED3 -> LED8
- LED17 pad 2: LED44 -> LED41
- LED17 pad 4: LED43 -> LED40
- LED18 pad 2: LED29 -> LED32
- LED18 pad 4: LED28 -> LED31
- LED19 pad 2: LED20 -> LED17
- LED19 pad 4: LED19 -> LED16
- LED2 pad 2: LED25 -> LED36
- LED2 pad 4: LED24 -> LED35
- LED20 pad 2: LED5 -> LED8
- LED20 pad 4: LED4 -> LED7
- LED21 pad 2: LED43 -> LED42
- LED21 pad 4: LED42 -> LED41
- LED22 pad 2: LED30 -> LED31
- LED22 pad 4: LED29 -> LED30
- LED23 pad 2: LED19 -> LED18
- LED23 pad 4: LED18 -> LED17
- LED24 pad 2: LED6 -> LED7
- LED24 pad 4: LED5 -> LED6
- LED25 pad 2: LED42 -> LED43
- LED25 pad 4: LED41 -> LED42
- LED26 pad 2: LED31 -> LED30
- LED26 pad 4: LED30 -> LED29
- LED27 pad 2: LED18 -> LED19
- LED27 pad 4: LED17 -> LED18
- LED28 pad 2: LED7 -> LED6
- LED28 pad 4: LED6 -> LED5
- LED29 pad 2: LED41 -> LED44
- LED29 pad 4: LED40 -> LED43
- LED3 pad 2: LED24 -> LED13
- LED3 pad 4: LED23 -> LED12
- LED30 pad 2: LED32 -> LED29
- LED30 pad 4: LED31 -> LED28
- LED31 pad 2: LED17 -> LED20
- LED31 pad 4: LED16 -> LED19
- LED32 pad 2: LED8 -> LED5
- LED32 pad 4: LED7 -> LED4
- LED33 pad 2: LED40 -> LED45
- LED33 pad 4: LED39 -> LED44
- LED34 pad 2: LED33 -> LED28
- LED34 pad 4: LED32 -> LED27
- LED35 pad 2: LED16 -> LED21
- LED35 pad 4: LED15 -> LED20
- LED36 pad 2: LED9 -> LED4
- LED36 pad 4: LED8 -> LED3
- LED37 pad 2: LED39 -> LED46
- LED37 pad 4: LED38 -> LED45
- LED38 pad 2: LED34 -> LED27
- LED38 pad 4: LED33 -> LED26
- LED39 pad 2: LED15 -> LED22
- LED39 pad 4: LED14 -> LED21
- LED4 pad 2: LED1 -> LED12
- LED4 pad 4: LED0 -> LED11
- LED40 pad 2: LED10 -> LED3
- LED40 pad 4: LED9 -> LED2
- LED41 pad 2: LED38 -> LED47
- LED41 pad 4: LED37 -> LED46
- LED42 pad 2: LED35 -> LED26
- LED42 pad 4: LED34 -> LED25
- LED43 pad 2: LED14 -> LED23
- LED43 pad 4: LED13 -> LED22
- LED44 pad 2: LED11 -> LED2
- LED44 pad 4: LED10 -> LED1
- LED45 pad 2: LED37 -> LED48
- LED45 pad 4: LED36 -> LED47
- LED46 pad 2: LED36 -> LED25
- LED46 pad 4: LED35 -> LED24
- LED47 pad 2: LED13 -> LED24
- LED47 pad 4: LED12 -> LED23
- LED48 pad 2: LED12 -> LED1
- LED48 pad 4: LED11 -> LED0
- LED5 pad 2: LED47 -> LED38
- LED5 pad 4: LED46 -> LED37
- LED6 pad 2: LED26 -> LED35
- LED6 pad 4: LED25 -> LED34
- LED7 pad 2: LED23 -> LED14
- LED7 pad 4: LED22 -> LED13
- LED8 pad 2: LED2 -> LED11
- LED8 pad 4: LED1 -> LED10
- LED9 pad 2: LED46 -> LED39
- LED9 pad 4: LED45 -> LED38
Routing:
- net LED0: track 149.1 -> 58.5 mm
- net COL6: track 254.9 -> 185.6 mm, vias 0 -> 6
- net ROW0: track 214.6 -> 281.1 mm, vias 0 -> 15
- net COL5: track 284.5 -> 222.9 mm, vias 2 -> 6
- net ROW1: track 206.2 -> 262.1 mm, vias 0 -> 16
- net COL11: track 62.9 -> 118.8 mm, vias 0 -> 6
- net COL1: track 342.5 -> 287.3 mm, vias 8 -> 6
- net LED46: track 65.1 -> 14.0 mm, vias 4 -> 0
- net ROW3: track 188.4 -> 238.0 mm, vias 0 -> 14
- net ROW2: track 208.2 -> 256.2 mm, vias 0 -> 16
- net COL4: track 272.6 -> 226.3 mm, vias 2 -> 6
- net LED11: track 58.2 -> 14.3 mm, vias 8 -> 0
- net COL7: track 235.2 -> 201.6 mm, vias 4 -> 6
- net COL8: track 210.1 -> 180.2 mm, vias 4 -> 6
- net VCC: track 1267.6 -> 1239.8 mm, vias 35 -> 51
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Other:
- board size 255 x 72 mm -> 262 x 72 mm
